File: DRIVER ROBOT.kicad_pcb (KiCad board)
At the start: 2 copper layers, 126 parts, among them IC1 BTS7960B, IC2 BTS7960B, IC3 BTS7960B, IC4 BTS7960B, IC5 BTS7960B, IC6 BTS7960B, J1 Screw_Terminal, J2 OUT MOTOR 1, J3 OUT MOTOR 2, J7 USB_C_Receptacle_USB2.0_16P, U1 AMS1117-3.3, U2 ESP32-WROOM-32U, U4 CH340C

Commit message: Schematic V1
Parts:
- removed the C10 at (116.9, 123.6)
- removed the C10 at (229.2, 129.5)
- removed the C10 at (159.5, 158.0)
- removed the C12 at (159.5, 161.0)
- removed the C12 at (229.2, 132.5)
- removed the C14 at (184.3, 72.0)
- removed the C14 at (206.8, 158.0)
- removed the C15 at (229.2, 135.5)
- removed the C15 at (183.5, 58.1)
- removed the C16 at (183.5, 61.6)
- removed the C16 at (229.2, 138.5)
- removed C18: 100nF, Capacitor_SMD:C_0805_2012Metric_Pad1.18x1.45mm_HandSolder
- removed C19: 0.1uF, Capacitor_SMD:C_0805_2012Metric_Pad1.18x1.45mm_HandSolder
- removed the C26 at (170.7, 134.7)
- removed the C26 at (162.4, 130.1)
- removed the C27 at (170.7, 137.7)
- removed the C27 at (162.4, 133.1)
- removed the C28 at (170.7, 140.7)
- removed the C28 at (162.4, 136.1)
- removed the C29 at (162.4, 139.1)
- removed the C29 at (170.7, 143.7)
- removed the C3 at (135.4, 117.3)
- removed the C3 at (159.5, 151.9)
- removed the C3 at (229.2, 123.4)
- removed C30: 10u, Capacitor_SMD:C_0805_2012Metric
- removed the C4 at (135.4, 120.3)
- removed the C4 at (206.8, 152.0)
- removed the C7 at (229.2, 126.4)
- removed the C7 at (159.5, 155.0)
- removed the IC3 at (150.1, 156.6)
- removed the IC3 at (219.9, 128.1)
- removed the IC4 at (219.9, 140.5)
- removed the IC4 at (150.1, 169.0)
- removed IC5, IC6: BTS7960B, Package_TO_SOT_SMD:TO-263-7_TabPin8
- removed L1: 15uH, Inductor_SMD:L_Chilisin_BMRx00060630
- removed OK1, OK3: HCPL2630, Package_SO:SOP-8_6.605x9.655mm_P2.54mm
- removed the R10 at (179.8, 127.8)
- removed the R10 at (137.0, 154.9)
- removed the R10 at (206.8, 126.4)
- removed the R11 at (206.8, 129.3)
- removed the R11 at (137.0, 157.8)
- removed the R11 at (180.4, 118.4)
- removed the R12 at (137.0, 160.8)
- removed the R12 at (180.4, 121.8)
- removed the R12 at (206.8, 132.3)
- removed the R13 at (137.0, 163.7)
- removed the R13 at (206.8, 135.2)
- removed the R13 at (116.9, 129.4)
- removed the R14 at (137.0, 166.7)
- removed the R14 at (206.8, 138.2)
- removed the R14 at (116.9, 133.4)
- removed the R15 at (206.8, 141.1)
- removed the R15 at (116.9, 137.5)
- removed the R15 at (137.0, 169.6)
- removed the R16 at (137.0, 172.6)
- removed the R16 at (116.9, 141.5)
- removed the R16 at (206.8, 144.1)
- removed the R23 at (148.1, 121.2)
- removed the R23 at (223.2, 115.8)
- removed the R24 at (137.0, 175.5)
- removed the R24 at (206.8, 147.0)
- removed the R24 at (148.1, 124.2)
- removed R55: 100k, Resistor_SMD:R_0805_2012Metric_Pad1.20x1.40mm_HandSolder
- removed R56: 24.9k, Resistor_SMD:R_0805_2012Metric_Pad1.20x1.40mm_HandSolder
- removed R57: 40.2k, Resistor_SMD:R_0805_2012Metric_Pad1.20x1.40mm_HandSolder
- removed the R7 at (134.6, 103.7)
- removed the R7 at (211.6, 152.0)
- removed the R9 at (206.8, 123.4)
- removed the R9 at (179.8, 124.9)
- removed the R9 at (137.0, 151.9)
- added C10: 100nF, Capacitor_SMD:C_0805_2012Metric_Pad1.18x1.45mm_HandSolder, F.Cu at (208.1, 60.4)
- added C12: 100nF, Capacitor_SMD:C_0805_2012Metric_Pad1.18x1.45mm_HandSolder, F.Cu at (167.7, 117.4)
- added C14: 470nF, Capacitor_SMD:C_0805_2012Metric_Pad1.18x1.45mm_HandSolder, F.Cu at (137.4, 93.2)
- added C15: 470nF, Capacitor_SMD:C_0805_2012Metric_Pad1.18x1.45mm_HandSolder, F.Cu at (208.1, 66.4)
- added C16: 470nF, Capacitor_SMD:C_0805_2012Metric_Pad1.18x1.45mm_HandSolder, F.Cu at (208.1, 69.4)
- added C26: 10uF, Capacitor_SMD:C_0805_2012Metric, F.Cu at (232.4, 99.6)
- added C27: 100nF, Capacitor_SMD:C_0805_2012Metric_Pad1.18x1.45mm_HandSolder, F.Cu at (237.0, 90.6)
- added C28: 10uF, Capacitor_SMD:C_0805_2012Metric, F.Cu at (232.4, 102.7)
- added C29: 100nF, Capacitor_SMD:C_0805_2012Metric_Pad1.18x1.45mm_HandSolder, F.Cu at (237.0, 93.6)
- added C3: 100nF, Capacitor_SMD:C_0805_2012Metric_Pad1.18x1.45mm_HandSolder, F.Cu at (208.1, 54.4)
- added C4: 470nF, Capacitor_SMD:C_0805_2012Metric_Pad1.18x1.45mm_HandSolder, F.Cu at (126.5, 70.3)
- added C6: 470uF 25V, Capacitor_SMD:CP_Elec_10x10.5, F.Cu at (123.7, 89.3)
- added C7: 470nF, Capacitor_SMD:C_0805_2012Metric_Pad1.18x1.45mm_HandSolder, F.Cu at (208.1, 57.4)
- added C8: 470uF 25V, Capacitor_SMD:CP_Elec_10x10.5, F.Cu at (193.0, 86.0)
- added D1: B5819W, Diode_SMD:Nexperia_CFP3_SOD-123W, F.Cu at (153.9, 97.5)
- added D18: SS34, Diode_SMD:D_SMA, F.Cu at (247.1, 105.5)
- added D2: LED, LED_SMD:LED_1206_3216Metric_Pad1.42x1.75mm_HandSolder, F.Cu at (249.0, 80.9)
- added D3: LED, LED_SMD:LED_1206_3216Metric_Pad1.42x1.75mm_HandSolder, F.Cu at (247.6, 96.8)
- added D4: LED, LED_SMD:LED_1206_3216Metric_Pad1.42x1.75mm_HandSolder, F.Cu at (128.5, 112.4)
- added D5: LED, LED_SMD:LED_1206_3216Metric_Pad1.42x1.75mm_HandSolder, F.Cu at (128.5, 114.8)
- added D6: LED, LED_SMD:LED_1206_3216Metric_Pad1.42x1.75mm_HandSolder, F.Cu at (213.5, 65.8)
- added D7: LED, LED_SMD:LED_1206_3216Metric_Pad1.42x1.75mm_HandSolder, F.Cu at (213.5, 69.2)
- added D8: LED, LED_SMD:LED_1206_3216Metric_Pad1.42x1.75mm_HandSolder, F.Cu at (247.6, 100.2)
- added H1: MountingHole, MountingHole:MountingHole_3.2mm_M3_DIN965_Pad_TopBottom, F.Cu at (103.0, 73.0)
- added H2: MountingHole, MountingHole:MountingHole_3.2mm_M3_DIN965_Pad_TopBottom, F.Cu at (103.0, 105.0)
- added H3: MountingHole, MountingHole:MountingHole_3.2mm_M3_DIN965_Pad_TopBottom, F.Cu at (175.0, 73.0)
- added H4: MountingHole, MountingHole:MountingHole_3.2mm_M3_DIN965_Pad_TopBottom, F.Cu at (175.0, 105.0)
- added IC3: BTS7960B, Package_TO_SOT_SMD:TO-263-7_TabPin8, F.Cu at (163.7, 74.7)
- added IC4: BTS7960B, Package_TO_SOT_SMD:TO-263-7_TabPin8, F.Cu at (198.7, 71.4)
- added J4: OLED 3 INCH, Connector_PinHeader_1.00mm:PinHeader_1x04_P1.00mm_Vertical, F.Cu at (197.7, 104.8)
- added Q1: SS8050, Package_TO_SOT_SMD:SOT-23_Handsoldering, F.Cu at (164.4, 85.4)
- added Q2: SS8050, Package_TO_SOT_SMD:SOT-23_Handsoldering, F.Cu at (164.3, 90.6)
- added R10: 10K, Resistor_SMD:R_0805_2012Metric_Pad1.20x1.40mm_HandSolder, F.Cu at (208.0, 75.3)
- added R11: 10K, Resistor_SMD:R_0805_2012Metric_Pad1.20x1.40mm_HandSolder, F.Cu at (208.0, 78.3)
- added R12: 470, Resistor_SMD:R_0805_2012Metric_Pad1.20x1.40mm_HandSolder, F.Cu at (208.0, 81.2)
- added R13: 510, Resistor_SMD:R_0805_2012Metric_Pad1.20x1.40mm_HandSolder, F.Cu at (208.0, 84.2)
- added R14: 10K, Resistor_SMD:R_0805_2012Metric_Pad1.20x1.40mm_HandSolder, F.Cu at (212.8, 72.4)
- added R15: 10K, Resistor_SMD:R_0805_2012Metric_Pad1.20x1.40mm_HandSolder, F.Cu at (212.8, 75.3)
- added R16: 470, Resistor_SMD:R_0805_2012Metric_Pad1.20x1.40mm_HandSolder, F.Cu at (212.8, 78.3)
- added R23: 10K, Resistor_SMD:R_0805_2012Metric_Pad1.20x1.40mm_HandSolder, F.Cu at (126.5, 76.2)
- added R24: 10K, Resistor_SMD:R_0805_2012Metric_Pad1.20x1.40mm_HandSolder, F.Cu at (212.8, 81.2)
- added R52: 10K, Resistor_SMD:R_0805_2012Metric_Pad1.20x1.40mm_HandSolder, F.Cu at (156.8, 127.6)
- added R7: 470, Resistor_SMD:R_0805_2012Metric_Pad1.20x1.40mm_HandSolder, F.Cu at (126.5, 72.2)
- added R9: 510, Resistor_SMD:R_0805_2012Metric_Pad1.20x1.40mm_HandSolder, F.Cu at (208.0, 72.4)
- added SW1: RST, Button_Switch_SMD:SW_SPST_CK_RS282G05A3, F.Cu at (159.8, 115.4)
- added SW3: BOOT, Button_Switch_SMD:SW_SPST_CK_RS282G05A3, F.Cu at (159.8, 120.6)
- added U3: HCPL-2630, Package_SO:SOP-8_6.605x9.655mm_P2.54mm, F.Cu at (143.3, 75.5)
- added U5: HCPL-2630, Package_SO:SOP-8_6.605x9.655mm_P2.54mm, F.Cu at (217.1, 58.5)
- C11: value 470uF -> 470nF; footprint Capacitor_THT:CP_Radial_D10.0mm_P2.50mm -> Capacitor_SMD:C_0805_2012Metric_Pad1.18x1.45mm_HandSolder
- C17: value 220nF -> 100nF
- C5: value 470uF -> 100nF; footprint Capacitor_THT:CP_Radial_D10.0mm_P2.50mm -> Capacitor_SMD:C_0805_2012Metric_Pad1.18x1.45mm_HandSolder
- J1: value Screw_Terminal -> INPUT 12V; footprint Connector_AMASS:AMASS_XT60PW-F_1x02_P7.20mm_Horizontal -> Connector_AMASS:AMASS_XT60-F_1x02_P7.20mm_Vertical
- R25, R26, R31, R32: value 10K -> 1k
- R27, R28, R29, R30: value 10K -> 330
- R33: value 100k -> 10K
- U2: moved to B.Cu
- moved J2 133.5 mm to (110.8, 86.7), turned to -90 degrees
- moved IC2 130.6 mm to (114.1, 75.0), turned to 180 degrees
- moved IC1 110.9 mm to (113.4, 103.0), turned to 180 degrees
- moved L2 98.1 mm to (239.6, 99.2)
- moved C13 95.0 mm to (137.4, 90.2)
- moved C24 94.4 mm to (237.0, 87.6)
- moved C11 90.8 mm to (208.1, 63.4)
- moved C25 87.2 mm to (232.4, 96.6)
- moved C21 85.7 mm to (232.4, 87.6)
- moved C23 85.7 mm to (232.4, 93.6)
- moved C22 85.7 mm to (232.4, 90.6)
- moved R22 85.3 mm to (227.8, 87.6)
- moved R58 83.3 mm to (227.8, 90.5)
- moved U1 81.4 mm to (244.3, 90.3)
- moved R63 74.4 mm to (227.8, 93.5)
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Connections:
- C1 pad 1: /MOTOR 1/ADC 1 -> Net-(IC1-IS)
- C11 pad 1: +12V -> Net-(IC4-IS)
- C17 pad 1: /ADC 4 -> EN
- C5 pad 1: +12V -> EN
- IC1 pad 4: /MOTOR 1/OUT 1 -> OUT 1
- IC1 pad 6: /MOTOR 1/ADC 1 -> Net-(IC1-IS)
- IC1 pad 8: /MOTOR 1/OUT 1 -> OUT 1
- IC2 pad 4: /MOTOR 1/OUT 2 -> OUT 2
- IC2 pad 6: /MOTOR 1/ADC 1 -> Net-(IC2-IS)
- IC2 pad 8: /MOTOR 1/OUT 2 -> OUT 2
- J2 pad 1: /OUT 2 -> OUT 2
- J2 pad 2: /OUT 1 -> OUT 1
- J3 pad 1: /OUT 4 -> OUT 4
- J3 pad 2: /OUT 3 -> OUT 3
- R1 pad 1: /MOTOR 1/PWM 1 -> /MOTOR 1/PWM_1
- R2 pad 1: /MOTOR 1/DIR 1 -> +5V
- R25 pad 1: /PWM_3 -> /MOTOR 1/PWM_1
- R25 pad 2: Net-(IC5-IN) -> +5V
- R26 pad 1: /ENA 3 -> /MOTOR 1/PWM_2
- R26 pad 2: Net-(IC5-INH) -> +5V
- R27 pad 1: /ADC 3 -> Net-(U3-C1)
- R27 pad 2: GND -> DIR1
- R28 pad 2: GND -> DIR2
- R29 pad 1: /PWM_4 -> Net-(U5-C1)
- R29 pad 2: Net-(IC6-IN) -> DIR3
- R3 pad 1: /MOTOR 1/ADC 1 -> Net-(IC1-IS)
- R30 pad 1: /ENA 4 -> Net-(U5-C2)
- R30 pad 2: Net-(IC6-INH) -> DIR4
- R31 pad 1: /ADC 4 -> /MOTOR 2/PWM_3
- R31 pad 2: GND -> +5V
- R32 pad 1: Net-(IC6-SR) -> /MOTOR 2/PWM_4
- R32 pad 2: GND -> +5V
- R33 pad 1: Net-(MP1584-EN) -> EN
- R33 pad 2: +5V -> +3V3
- R5 pad 1: /MOTOR 1/PWM 1 -> /MOTOR 1/PWM_2
- R6 pad 1: /MOTOR 1/DIR 2 -> +5V
- U1 pad 2: /3V3 -> +3V3
- U2 pad 10: unconnected-(U2-IO25-Pad10) -> /ESP32/DIR1
- U2 pad 11: unconnected-(U2-IO26-Pad11) -> /ESP32/DIR2
- U2 pad 12: unconnected-(U2-IO27-Pad12) -> /ESP32/PWM 1
- U2 pad 13: unconnected-(U2-IO14-Pad13) -> /ESP32/PWM 2
- U2 pad 2: /3V3 -> +3V3
- U2 pad 33: unconnected-(U2-IO21-Pad33) -> /SDA
- U2 pad 36: unconnected-(U2-IO22-Pad36) -> /SCL
- U2 pad 8: unconnected-(U2-IO32-Pad8) -> /ESP32/DIR 3
- U2 pad 9: unconnected-(U2-IO33-Pad9) -> /ESP32/DIR 4
- U4 pad 16: /3V3 -> +3V3
Other:
- board outline added: 80 x 40 mm

Commit message: Schematic V1.1
Parts:
- added SW4: BOOT, Button_Switch_THT:SW_E-Switch_EG1224_SPDT_Angled, F.Cu at (149.1, 104.6)
- C1, C2, C4, C9, IC1, IC2, IC3, IC4, R1, R2, R23, R25, R26, R27, R28, R3, R4, R5, R6, R7, R8, U3: moved to B.Cu
- J1: footprint Connector_AMASS:AMASS_XT60-F_1x02_P7.20mm_Vertical -> TerminalBlock_Phoenix:TerminalBlock_Phoenix_MKDS-1,5-2_1x02_P5.00mm_Horizontal
- SW1, SW3: footprint Button_Switch_SMD:SW_SPST_CK_RS282G05A3 -> Button_Switch_SMD:SW_SPST_FSMSM
- U2: moved to F.Cu
- moved D9 48.9 mm to (143.7, 97.5), turned to 180 degrees
- moved U2 48.0 mm to (119.9, 98.4), turned to 180 degrees
- moved IC4 46.9 mm to (152.0, 75.6), turned to 90 degrees
- moved R1 37.8 mm to (126.0, 70.1)
- moved R25 37.8 mm to (129.8, 70.1)
- moved C4 37.4 mm to (126.5, 107.7)
- moved R2 33.9 mm to (126.0, 72.0)
- moved R7 33.5 mm to (126.5, 105.7)
- moved J3 30.1 mm to (173.7, 93.5), turned to 90 degrees
- moved R4 30.0 mm to (126.0, 74.0)
- moved R8 29.5 mm to (126.5, 103.8)
- moved IC1 27.4 mm to (112.0, 75.6), turned to 90 degrees
- moved C2 26.0 mm to (126.0, 76.0)
- moved R23 25.6 mm to (126.5, 101.8)
- moved IC3 24.7 mm to (139.0, 75.6), turned to 90 degrees
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Connections:
- U2 pad 10: /ESP32/DIR1 -> DIR1
- U2 pad 11: /ESP32/DIR2 -> DIR2
- U2 pad 12: /ESP32/PWM 1 -> PWM1
- U2 pad 13: /ESP32/PWM 2 -> PWM2
- U2 pad 8: /ESP32/DIR 3 -> DIR3
- U2 pad 9: /ESP32/DIR 4 -> DIR4

Commit message: layout v1
Parts:
- moved U2 39.9 mm to (80.8, 106.2)
- moved IC3 26.4 mm to (165.4, 75.0), turned to 0 degrees
- moved IC4 18.1 mm to (165.4, 87.7), turned to 0 degrees
- moved IC2 16.9 mm to (113.1, 86.8), turned to 180 degrees
- moved R23 13.8 mm to (126.0, 88.0)
- moved C4 13.8 mm to (126.0, 93.9)
- moved C9 13.8 mm to (126.0, 86.0)
- moved R5 13.8 mm to (126.0, 82.0)
- moved R6 13.8 mm to (126.0, 84.0)
- moved R7 13.8 mm to (126.0, 91.9)
- moved R8 13.8 mm to (126.0, 90.0)
- moved R26 13.8 mm to (129.7, 82.0)
- moved J3 8.50 mm to (173.7, 85.0)
- moved J2 8.00 mm to (103.8, 80.0)
- moved IC1 1.29 mm to (113.1, 75.0), turned to 180 degrees
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