File: DRIVER ROBOT.kicad_pcb (KiCad board)
At the start: 2 copper layers, 80 x 30 mm, 102 parts, among them IC1 BTS7960B, IC2 BTS7960B, IC3 BTS7960B, IC4 BTS7960B, J1 INPUT 12V, J2 OUT MOTOR 1, J3 OUT MOTOR 2, J4 OLED 3 INCH, J7 USB_C_Receptacle_USB2.0_16P, Q1 SS8050, Q2 SS8050, SW1 RST, SW3 BOOT, U1 AMS1117-3.3, U2 ESP32-WROOM-32U, U3 HCPL-2630, U4 CH340C, U5 HCPL-2630

Commit message: layout v2
Parts:
- removed J7: USB_C_Receptacle_USB2.0_16P, Connector_USB:USB_C_Receptacle_GCT_USB4105-xx-A_16P_TopMnt_Horizontal
- added J5: USB_C_Receptacle_USB2.0_14P, Connector_USB:USB_C_Plug_ShenzhenJingTuoJin_918-118A2021Y40002_Vertical, F.Cu at (164.6, 95.3)
- C1, C10, C11, C12, C13, C14, C17, C2, C20, C3, C4, C5, C7, C9: footprint Capacitor_SMD:C_0805_2012Metric_Pad1.18x1.45mm_HandSolder -> Capacitor_SMD:C_0603_1608Metric_Pad1.08x0.95mm_HandSolder
- C15, C16: footprint Capacitor_SMD:C_0805_2012Metric_Pad1.18x1.45mm_HandSolder -> Capacitor_SMD:C_0603_1608Metric_Pad1.08x0.95mm_HandSolder; moved to F.Cu
- C23: footprint Capacitor_SMD:C_0805_2012Metric -> Capacitor_SMD:C_0603_1608Metric_Pad1.08x0.95mm_HandSolder
- D8: footprint LED_SMD:LED_0805_2012Metric_Pad1.15x1.40mm_HandSolder -> LED_SMD:LED_0603_1608Metric_Pad1.05x0.95mm_HandSolder
- R1, R10, R11, R12, R13, R14, R15, R16, R17, R18, R19, R2, R20, R21, R22, R25, R26, R27, R28, R29, R3, R30, R31, R32, R33, R4, R5, R52, R58, R6, R63, R64, R7, R71, R8, R9: footprint Resistor_SMD:R_0805_2012Metric_Pad1.20x1.40mm_HandSolder -> Resistor_SMD:R_0603_1608Metric_Pad0.98x0.95mm_HandSolder
- R23, R24: moved to F.Cu
- moved C15 25.5 mm to (169.2, 76.7), turned to 0 degrees
- moved R24 22.8 mm to (169.2, 74.7), turned to 0 degrees
- moved R23 21.5 mm to (108.5, 74.9)
- moved C16 15.9 mm to (156.3, 82.6)
- moved R18 6.52 mm to (163.9, 98.0), turned to 180 degrees
- moved D1 6.29 mm to (160.7, 93.3), turned to 0 degrees
- moved R17 3.03 mm to (164.8, 93.3)
- moved R15 2.82 mm to (152.4, 91.2)
- moved R14 2.38 mm to (152.4, 89.7)
- moved Q1 2.28 mm to (156.4, 87.2)
- moved R19 2.18 mm to (160.3, 98.0)
- moved C27 1.61 mm to (147.7, 72.6)
- moved R65 1.32 mm to (151.8, 83.2)
- moved D3 1.32 mm to (151.8, 85.2)
- moved C26 1.31 mm to (151.9, 81.2)
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Connections:
- J4 pad 1: +12V -> +3V3
Routing:
- net +12V: track 0.00 -> 128.8 mm, vias 0 -> 4
- net +5V: track 0.00 -> 112.9 mm, vias 0 -> 4
- net +3V3: track 0.00 -> 84.9 mm
- net IO0: track 0.00 -> 56.6 mm, vias 0 -> 1
- net TXD: track 0.00 -> 55.6 mm
- net RXD: track 0.00 -> 52.8 mm
- net UD-: track 0.00 -> 34.5 mm, vias 0 -> 3
- net UD+: track 0.00 -> 34.1 mm
- net DIR2: track 0.00 -> 31.7 mm, vias 0 -> 1
- net PWM1: track 0.00 -> 28.9 mm, vias 0 -> 1
- net /MOTOR 2/PWM_4: track 0.00 -> 25.7 mm
- net OUT 1: track 0.00 -> 25.4 mm
- net OUT 2: track 0.00 -> 24.4 mm
- net OUT 4: track 0.00 -> 24.0 mm
- net OUT 3: track 0.00 -> 23.1 mm
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- added copper zone on B.Cu, net GND
- added copper zone on F.Cu, net GND
- added copper zone on F.Cu, net Net-(D9-A)
- added copper zone on B.Cu, net OUT 1
- added copper zone on B.Cu, net OUT 2
- added copper zone on B.Cu, net OUT 3
- added copper zone on B.Cu, net OUT 4

Commit message: layout final v1
Parts:
- moved C15 0.49 mm to (169.2, 77.2)
- moved R11 0.42 mm to (152.4, 79.8)
- moved C29 0.05 mm to (147.7, 77.0)
Routing:
- net +3V3: track 84.9 -> 118.0 mm, vias 0 -> 4
- net /MOTOR 2/PWM_4: track 25.7 -> 27.2 mm
- net PWM2: track 13.0 -> 12.0 mm
- net Net-(IC3-IN): track 6.25 -> 5.50 mm
- net ~{DTR}: track 17.1 -> 17.7 mm
- net GND: vias 16 -> 25

Commit message: layout final v2
Parts:
- moved H2 1.61 mm to (102.0, 96.0)
- moved H4 1.60 mm to (175.9, 95.9)
- moved H1 1.33 mm to (102.1, 72.1)
- moved H3 1.33 mm to (175.9, 72.1)
Changed lines of the file:
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@@
 	(footprint "MountingHole:MountingHole_3.2mm_M3_DIN965_Pad_TopBottom"
 		(layer "F.Cu")
-		(at 103 94.65)
+		(at 102.05 95.95)
 		(descr "Mounting Hole 3.2mm, M3, generated by kicad-footprint-generator mountinghole.py")
 		(tags "mountinghole M3 DIN965")
@@
 	(footprint "MountingHole:MountingHole_3.2mm_M3_DIN965_Pad_TopBottom"
 		(layer "F.Cu")
-		(at 103 73)
+		(at 102.06 72.06)
 		(descr "Mounting Hole 3.2mm, M3, generated by kicad-footprint-generator mountinghole.py")
 		(tags "mountinghole M3 DIN965")
@@
 	(footprint "MountingHole:MountingHole_3.2mm_M3_DIN965_Pad_TopBottom"
 		(layer "F.Cu")
-		(at 175 94.65)
+		(at 175.94 95.94)
 		(descr "Mounting Hole 3.2mm, M3, generated by kicad-footprint-generator mountinghole.py")
 		(tags "mountinghole M3 DIN965")
@@
 	(footprint "MountingHole:MountingHole_3.2mm_M3_DIN965_Pad_TopBottom"
 		(layer "F.Cu")
-		(at 175 73)
+		(at 175.94 72.06)
 		(descr "Mounting Hole 3.2mm, M3, generated by kicad-footprint-generator mountinghole.py")
 		(tags "mountinghole M3 DIN965")

Commit message: layout final v3
Parts:
- added G***: LOGO, LOGO, F.Cu at (113.9, 84.8)
- D2, D3: footprint LED_SMD:LED_0805_2012Metric_Pad1.15x1.40mm_HandSolder -> LED_SMD:LED_0603_1608Metric_Pad1.05x0.95mm_HandSolder
- moved D8 7.48 mm to (124.1, 88.2)
- moved R71 5.74 mm to (128.1, 86.8), turned to 180 degrees
- moved L2 5.29 mm to (125.9, 81.4), turned to 90 degrees
- moved C23 4.43 mm to (131.4, 78.2), turned to 0 degrees
- moved C13 4.29 mm to (125.3, 93.6)
- moved C14 3.79 mm to (125.3, 92.1)
- moved D18 3.72 mm to (125.5, 74.4)
- moved C4 3.32 mm to (125.3, 90.6)
- moved R69 3.15 mm to (130.5, 73.3)
- moved R22 3.12 mm to (134.8, 78.2), turned to 0 degrees
- moved R7 2.85 mm to (125.3, 89.0)
- moved C24 2.69 mm to (132.6, 73.3), turned to 90 degrees
- moved R25 2.50 mm to (135.0, 73.0)
- moved R26 2.50 mm to (131.1, 73.0)
- moved R27 2.50 mm to (134.9, 86.6)
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Connections:
- J4 pad 1: +3V3 -> /SDA
- J4 pad 2: /SDA -> /SCL
- J4 pad 3: /SCL -> GND
- J4 pad 4: GND -> +3V3
Routing:
- net +12V: track 128.3 -> 13.1 mm
- net DIR2: track 31.7 -> 22.4 mm
- net +5V: track 112.8 -> 121.5 mm
- net PWM1: track 28.9 -> 22.0 mm
- net +3V3: track 118.0 -> 114.3 mm
- net DIR3: track 7.49 -> 3.81 mm
- net /MOTOR 2/PWM_3: track 14.0 -> 10.6 mm
- net DIR1: track 15.1 -> 18.0 mm
- net Net-(MP1584-EN): track 6.53 -> 9.43 mm
- net /SCL: track 3.13 -> 5.87 mm
- net Net-(MP1584-SW): track 19.5 -> 16.8 mm
- net Net-(IC2-IS): track 7.95 -> 5.34 mm
- net Net-(IC2-SR): track 7.56 -> 5.25 mm
- net Net-(MP1584-COMP): track 3.90 -> 6.11 mm
- net /MOTOR 2/PWM_4: track 27.2 -> 25.2 mm
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- added copper zone on F.Cu, net +12V
Other:
- board text added: "+"
- board text added: "LEFT"
- board text added: "RIGHT"
