File: Motor 2.kicad_sch (KiCad schematic)
At the start: 20 parts, among them IC3 BTS7960B, IC4 BTS7960B

Commit message: Schematic V1
Parts:
- removed C12: 470nF, Capacitor_SMD:C_0805_2012Metric_Pad1.18x1.45mm_HandSolder, symbol Device:C
- added C11: 470nF, Capacitor_SMD:C_0805_2012Metric_Pad1.18x1.45mm_HandSolder, symbol Device:C
- added R29, R30: 330, Resistor_SMD:R_0805_2012Metric_Pad1.20x1.40mm_HandSolder, symbol Device:R
- added R31, R32: 1k, Resistor_SMD:R_0805_2012Metric_Pad1.20x1.40mm_HandSolder, symbol Device:R
- added U5: HCPL-2630, Package_SO:SOP-8_6.605x9.655mm_P2.54mm, symbol Isolator:HCPL-2630
- C8: value 10000uF 50v -> 470uF 25V; footprint (none) -> Capacitor_SMD:CP_Elec_10x10.5
- D6, D7: footprint (none) -> LED_SMD:LED_1206_3216Metric_Pad1.42x1.75mm_HandSolder
Connections:
- net DIR 4 is gone; now on net +5V: R14.1
- net GND: now also C11.2, U5.5 (GND)
- net OUT 3: no longer IC3.4 (OUT_1)
- net OUT 4: no longer IC4.4 (OUT_1), IC4.8 (OUT_2)
- net ADC 2: no longer names the net of IC4.6 (IS), R16.1
- net ADC 2: now also C11.1
- net ADC_2: no longer names the net of C7.1, IC3.6 (IS), R12.1
- net DIR 3 renamed +5V
- net +5V: now also R31.2, R32.2, U5.8 (VCC)
- net PWM 2 renamed PWM_3
- net PWM_3: now also R31.1, U5.7 (VO1); no longer R15.1
- new net: R30.1, U5.3 (C2)
- new net: R29.1, U5.2 (C1)
- new net DIR3: R29.2
- new net DIR4: R30.2
- new net OUT 1: IC3.4 (OUT_1)
- new net OUT 2: IC4.4 (OUT_1), IC4.8 (OUT_2)
- new net PWM2: U5.1 (A1), U5.4 (A2)
- new net PWM_4: R15.1, R32.1, U5.6 (VO2)
Other:
- title: Board Robot SUMO -> Board Robot SOCCER & SUMO

Commit message: layout v1.1
Parts:
- D6, D7: footprint LED_SMD:LED_1206_3216Metric_Pad1.42x1.75mm_HandSolder -> LED_SMD:LED_0805_2012Metric_Pad1.15x1.40mm_HandSolder
Connections:
- net OUT 1 is gone; now on net OUT 3: IC3.4 (OUT_1)
- net OUT 2 is gone; now on net OUT 4: IC4.4 (OUT_1), IC4.8 (OUT_2)
Changed lines of the file:
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@@
 		)
 	)
-	(label "OUT 2"
+	(label "OUT 4"
 		(at 209.55 96.52 180)
 		(effects
@@
 		)
 	)
-	(label "OUT 2"
+	(label "OUT 4"
 		(at 240.03 88.9 0)
 		(effects
@@
 		)
 	)
-	(label "OUT 1"
+	(label "OUT 3"
 		(at 137.16 96.52 180)
 		(effects
@@
 			)
 		)
-		(property "Footprint" "LED_SMD:LED_1206_3216Metric_Pad1.42x1.75mm_HandSolder"
+		(property "Footprint" "LED_SMD:LED_0805_2012Metric_Pad1.15x1.40mm_HandSolder"
 			(at 176.53 83.82 0)
 			(hide yes)
@@
 			)
 		)
-		(property "Footprint" "LED_SMD:LED_1206_3216Metric_Pad1.42x1.75mm_HandSolder"
+		(property "Footprint" "LED_SMD:LED_0805_2012Metric_Pad1.15x1.40mm_HandSolder"
 			(at 176.53 80.01 0)
 			(hide yes)

Commit message: layout v2
Parts:
- C10, C11, C15, C16, C3, C7: footprint Capacitor_SMD:C_0805_2012Metric_Pad1.18x1.45mm_HandSolder -> Capacitor_SMD:C_0603_1608Metric_Pad1.08x0.95mm_HandSolder
- R10, R11, R12, R13, R14, R15, R16, R29, R30, R31, R32, R9: footprint Resistor_SMD:R_0805_2012Metric_Pad1.20x1.40mm_HandSolder -> Resistor_SMD:R_0603_1608Metric_Pad0.98x0.95mm_HandSolder
Changed lines of the file:
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@@
 			)
 		)
-		(property "Footprint" "Resistor_SMD:R_0805_2012Metric_Pad1.20x1.40mm_HandSolder"
+		(property "Footprint" "Resistor_SMD:R_0603_1608Metric_Pad0.98x0.95mm_HandSolder"
 			(at 94.488 96.52 90)
 			(hide yes)
@@
 			)
 		)
-		(property "Footprint" "Resistor_SMD:R_0805_2012Metric_Pad1.20x1.40mm_HandSolder"
+		(property "Footprint" "Resistor_SMD:R_0603_1608Metric_Pad0.98x0.95mm_HandSolder"
 			(at 94.488 83.82 90)
 			(hide yes)
@@
 			)
 		)
-		(property "Footprint" "Capacitor_SMD:C_0805_2012Metric_Pad1.18x1.45mm_HandSolder"
+		(property "Footprint" "Capacitor_SMD:C_0603_1608Metric_Pad1.08x0.95mm_HandSolder"
 			(at 115.2652 115.57 0)
 			(hide yes)
@@
 			)
 		)
-		(property "Footprint" "Resistor_SMD:R_0805_2012Metric_Pad1.20x1.40mm_HandSolder"
+		(property "Footprint" "Resistor_SMD:R_0603_1608Metric_Pad0.98x0.95mm_HandSolder"
 			(at 195.072 86.36 90)
 			(hide yes)
@@
 			)
 		)
-		(property "Footprint" "Resistor_SMD:R_0805_2012Metric_Pad1.20x1.40mm_HandSolder"
+		(property "Footprint" "Resistor_SMD:R_0603_1608Metric_Pad0.98x0.95mm_HandSolder"
 			(at 106.172 111.76 90)
 			(hide yes)
@@
 			)
 		)
-		(property "Footprint" "Capacitor_SMD:C_0805_2012Metric_Pad1.18x1.45mm_HandSolder"
+		(property "Footprint" "Capacitor_SMD:C_0603_1608Metric_Pad1.08x0.95mm_HandSolder"
 			(at 199.0852 130.81 0)
 			(hide yes)
@@
 			)
 		)
-		(property "Footprint" "Resistor_SMD:R_0805_2012Metric_Pad1.20x1.40mm_HandSolder"
+		(property "Footprint" "Resistor_SMD:R_0603_1608Metric_Pad0.98x0.95mm_HandSolder"
 			(at 62.23 94.742 90)
 			(hide yes)
@@
 			)
 		)
-		(property "Footprint" "Capacitor_SMD:C_0805_2012Metric_Pad1.18x1.45mm_HandSolder"
+		(property "Footprint" "Capacitor_SMD:C_0603_1608Metric_Pad1.08x0.95mm_HandSolder"
 			(at 148.2852 129.54 0)
 			(hide yes)
@@
 			)
 		)
-		(property "Footprint" "Capacitor_SMD:C_0805_2012Metric_Pad1.18x1.45mm_HandSolder"
+		(property "Footprint" "Capacitor_SMD:C_0603_1608Metric_Pad1.08x0.95mm_HandSolder"
 			(at 197.8152 113.03 0)
 			(hide yes)
@@
 			)
 		)
-		(property "Footprint" "Resistor_SMD:R_0805_2012Metric_Pad1.20x1.40mm_HandSolder"
+		(property "Footprint" "Resistor_SMD:R_0603_1608Metric_Pad0.98x0.95mm_HandSolder"
 			(at 62.23 89.662 90)
 			(hide yes)
@@
 			)
 		)
-		(property "Footprint" "Resistor_SMD:R_0805_2012Metric_Pad1.20x1.40mm_HandSolder"
+		(property "Footprint" "Resistor_SMD:R_0603_1608Metric_Pad0.98x0.95mm_HandSolder"
 			(at 202.692 109.22 90)
 			(hide yes)
@@
 			)
 		)
-		(property "Footprint" "Capacitor_SMD:C_0805_2012Metric_Pad1.18x1.45mm_HandSolder"
+		(property "Footprint" "Capacitor_SMD:C_0603_1608Metric_Pad1.08x0.95mm_HandSolder"
 			(at 127.9652 115.57 0)
 			(hide yes)
@@
 			)
 		)
-		(property "Footprint" "Capacitor_SMD:C_0805_2012Metric_Pad1.18x1.45mm_HandSolder"
+		(property "Footprint" "Capacitor_SMD:C_0603_1608Metric_Pad1.08x0.95mm_HandSolder"
 			(at 185.1152 113.03 0)
 			(hide yes)
@@
 			)
 		)
-		(property "Footprint" "Resistor_SMD:R_0805_2012Metric_Pad1.20x1.40mm_HandSolder"
+		(property "Footprint" "Resistor_SMD:R_0603_1608Metric_Pad0.98x0.95mm_HandSolder"
 			(at 131.572 86.36 90)
 			(hide yes)
@@
 			)
 		)
-		(property "Footprint" "Resistor_SMD:R_0805_2012Metric_Pad1.20x1.40mm_HandSolder"
+		(property "Footprint" "Resistor_SMD:R_0603_1608Metric_Pad0.98x0.95mm_HandSolder"
 			(at 120.142 86.36 90)
 			(hide yes)
@@
 			)
 		)
-		(property "Footprint" "Resistor_SMD:R_0805_2012Metric_Pad1.20x1.40mm_HandSolder"
+		(property "Footprint" "Resistor_SMD:R_0603_1608Metric_Pad0.98x0.95mm_HandSolder"
 			(at 173.482 109.22 90)
 			(hide yes)
@@
 			)
 		)
-		(property "Footprint" "Resistor_SMD:R_0805_2012Metric_Pad1.20x1.40mm_HandSolder"
+		(property "Footprint" "Resistor_SMD:R_0603_1608Metric_Pad0.98x0.95mm_HandSolder"
 			(at 132.842 111.76 90)
 			(hide yes)
@@
 			)
 		)
-		(property "Footprint" "Resistor_SMD:R_0805_2012Metric_Pad1.20x1.40mm_HandSolder"
+		(property "Footprint" "Resistor_SMD:R_0603_1608Metric_Pad0.98x0.95mm_HandSolder"
 			(at 202.692 86.36 90)
 			(hide yes)

Commit message: layout final v6
Parts:
- removed IC3, IC4: BTS7960B, Package_TO_SOT_SMD:TO-263-7_TabPin8, symbol Driver BTN 2023 FIX-eagle-import:BTS7960B
- added Q7, Q8: BTN8982TA, Package_TO_SOT_SMD:TO-263-7_TabPin8, symbol Power_Management:BTN8982TA
Connections:
- net +12V: now also Q7.7, Q8.7
- net GND: now also Q7.1, Q8.1
- net OUT 3: now also Q7.4, Q7.8
- net OUT 4: now also Q8.4, Q8.8
- net at R15.2: now also Q8.2 (IN)
- net at R14.2: now also Q8.3 (INH)
- net at C10.1, R13.1: now also Q8.5 (SR)
- net at C11.1, R16.1: now also Q8.6 (IS)
- net at C3.1, R9.1: now also Q7.5 (SR)
- net at C7.1, R12.1: now also Q7.6 (IS)
- net at R11.2: now also Q7.2 (IN)
- net at R10.2: now also Q7.3 (INH)
Other:
- moved on the sheet: C10, C11, C3, C7, R10, R11, R12, R13, R14, R15, R16, R9
